File: hardware/ece129_discharger.kicad_pcb (KiCad board)
At the start: 2 copper layers, 0 parts

Commit message: initial layout, power traces remain
Parts:
- added C1: 100uF, Capacitor_SMD:C_0805_2012Metric_Pad1.18x1.45mm_HandSolder, F.Cu at (57.3, 56.6)
- added C10: 22uF (10V), Capacitor_SMD:C_0805_2012Metric_Pad1.18x1.45mm_HandSolder, F.Cu at (179.4, 156.4)
- added C11: 100nF, Capacitor_SMD:C_0805_2012Metric_Pad1.18x1.45mm_HandSolder, F.Cu at (179.4, 159.9)
- added C12: 100nF, Capacitor_SMD:C_0805_2012Metric_Pad1.18x1.45mm_HandSolder, F.Cu at (67.4, 154.8)
- added C2: 100uF, Capacitor_SMD:C_0805_2012Metric_Pad1.18x1.45mm_HandSolder, F.Cu at (65.5, 56.6)
- added C22: 0.22uF, Capacitor_SMD:C_0805_2012Metric_Pad1.18x1.45mm_HandSolder, F.Cu at (122.4, 61.1)
- added C23: 0.22uF, Capacitor_SMD:C_0805_2012Metric_Pad1.18x1.45mm_HandSolder, F.Cu at (113.4, 61.1)
- added C24: 4.7nF, Capacitor_SMD:C_0805_2012Metric_Pad1.18x1.45mm_HandSolder, F.Cu at (117.9, 61.1)
- added C25: 1uF, Capacitor_SMD:C_0805_2012Metric_Pad1.18x1.45mm_HandSolder, F.Cu at (112.4, 66.1)
- added C26: 47nF, Capacitor_SMD:C_0805_2012Metric_Pad1.18x1.45mm_HandSolder, F.Cu at (119.9, 80.0)
- added C27: 10nF, Capacitor_SMD:C_0805_2012Metric_Pad1.18x1.45mm_HandSolder, F.Cu at (110.4, 80.0)
- added C28: 0.1uF, Capacitor_SMD:C_0805_2012Metric_Pad1.18x1.45mm_HandSolder, F.Cu at (129.4, 72.1)
- added C29: 0.1uF, Capacitor_SMD:C_0805_2012Metric_Pad1.18x1.45mm_HandSolder, F.Cu at (129.4, 75.6)
- added C3: 100uF, Capacitor_SMD:C_0805_2012Metric_Pad1.18x1.45mm_HandSolder, F.Cu at (47.0, 56.9)
- added C30: 47nF, Capacitor_SMD:C_0805_2012Metric_Pad1.18x1.45mm_HandSolder, F.Cu at (179.4, 61.3)
- added C31: 10nF, Capacitor_SMD:C_0805_2012Metric_Pad1.18x1.45mm_HandSolder, F.Cu at (165.9, 74.3)
- added C32: 10uF, Capacitor_SMD:C_0805_2012Metric_Pad1.18x1.45mm_HandSolder, F.Cu at (174.4, 61.3)
- added C33: 1uF, Capacitor_SMD:C_0805_2012Metric_Pad1.18x1.45mm_HandSolder, F.Cu at (170.9, 61.3)
- added C34: 0.1uF, Capacitor_SMD:C_0805_2012Metric_Pad1.18x1.45mm_HandSolder, F.Cu at (146.1, 76.3)
- added C4: 100uF, Capacitor_SMD:C_0805_2012Metric_Pad1.18x1.45mm_HandSolder, F.Cu at (75.8, 56.5)
- added C5: 100uF, Capacitor_SMD:C_0805_2012Metric_Pad1.18x1.45mm_HandSolder, F.Cu at (56.7, 67.3)
- added C6: 100uF, Capacitor_SMD:C_0805_2012Metric_Pad1.18x1.45mm_HandSolder, F.Cu at (57.0, 98.1)
- added C7: 100uF, Capacitor_SMD:C_0805_2012Metric_Pad1.18x1.45mm_HandSolder, F.Cu at (56.8, 87.3)
- added C8: 100uF, Capacitor_SMD:C_0805_2012Metric_Pad1.18x1.45mm_HandSolder, F.Cu at (55.6, 77.3)
- added C9: 10uF (50V), Capacitor_SMD:C_0805_2012Metric_Pad1.18x1.45mm_HandSolder, F.Cu at (177.4, 144.4)
- added D1: 1N4007, Diode_THT:D_DO-41_SOD81_P10.16mm_Horizontal, F.Cu at (178.9, 120.9)
- added J1: Conn_01x03, Connector_Molex:Molex_Nano-Fit_105309-xx03_1x03_P2.50mm_Vertical, F.Cu at (85.2, 57.6)
- added J10: Conn_01x02, Connector_Molex:Molex_Nano-Fit_105309-xx02_1x02_P2.50mm_Vertical, F.Cu at (50.4, 73.6)
- added J11: Conn_02x05_Top_Bottom, Connector_Molex:Molex_Nano-Fit_105310-xx10_2x05_P2.50mm_Vertical, F.Cu at (82.7, 113.7)
- added J12: Conn_01x08, Connector_Molex:Molex_Nano-Fit_105309-xx08_1x08_P2.50mm_Vertical, F.Cu at (75.9, 141.3)
- added J13: Conn_02x05_Top_Bottom, Connector_Molex:Molex_Nano-Fit_105310-xx10_2x05_P2.50mm_Vertical, F.Cu at (170.4, 148.9)
- added J14: Conn_01x02, Connector_Molex:Molex_Nano-Fit_105309-xx02_1x02_P2.50mm_Vertical, F.Cu at (168.9, 50.6)
- added J16: Conn_01x08, Connector_Molex:Molex_Nano-Fit_105309-xx08_1x08_P2.50mm_Vertical, F.Cu at (68.9, 121.3)
- added J17: Conn_01x02, Connector_Molex:Molex_Nano-Fit_105309-xx02_1x02_P2.50mm_Vertical, F.Cu at (172.1, 111.3)
- added J18: Conn_01x02, Connector_Molex:Molex_Nano-Fit_105309-xx02_1x02_P2.50mm_Vertical, F.Cu at (178.5, 151.6)
- added J19: Conn_01x04, Connector_Molex:Molex_Nano-Fit_105309-xx04_1x04_P2.50mm_Vertical, F.Cu at (113.6, 48.7)
- added J2: Conn_01x02, Connector_Molex:Molex_Nano-Fit_105309-xx02_1x02_P2.50mm_Vertical, F.Cu at (87.9, 49.8)
- added J20: Conn_01x02, Connector_Molex:Molex_Nano-Fit_105309-xx02_1x02_P2.50mm_Vertical, F.Cu at (170.2, 139.2)
- added J3: Conn_01x02, Connector_Molex:Molex_Nano-Fit_105309-xx02_1x02_P2.50mm_Vertical, F.Cu at (60.3, 50.0)
- added J4: Conn_01x02, Connector_Molex:Molex_Nano-Fit_105309-xx02_1x02_P2.50mm_Vertical, F.Cu at (69.0, 50.0)
- added J5: Conn_01x02, Connector_Molex:Molex_Nano-Fit_105309-xx02_1x02_P2.50mm_Vertical, F.Cu at (50.5, 50.4)
- added J6: Conn_01x02, Connector_Molex:Molex_Nano-Fit_105309-xx02_1x02_P2.50mm_Vertical, F.Cu at (78.8, 50.0)
- added J7: Conn_01x02, Connector_Molex:Molex_Nano-Fit_105309-xx02_1x02_P2.50mm_Vertical, F.Cu at (50.2, 64.1)
- added J8: Conn_01x02, Connector_Molex:Molex_Nano-Fit_105309-xx02_1x02_P2.50mm_Vertical, F.Cu at (50.4, 94.8)
- added J9: Conn_01x02, Connector_Molex:Molex_Nano-Fit_105309-xx02_1x02_P2.50mm_Vertical, F.Cu at (50.3, 84.1)
- added Q2: AO3400A, Package_TO_SOT_SMD:SOT-23, F.Cu at (178.9, 106.2)
- added R1: 10k, Resistor_SMD:R_0805_2012Metric_Pad1.20x1.40mm_HandSolder, F.Cu at (60.3, 56.6)
- added R10: 56k, Resistor_SMD:R_0805_2012Metric_Pad1.20x1.40mm_HandSolder, F.Cu at (87.4, 89.2)
- added R11: 200k, Resistor_SMD:R_0805_2012Metric_Pad1.20x1.40mm_HandSolder, F.Cu at (83.9, 91.7)
- added R12: 10k, Resistor_SMD:R_0805_2012Metric_Pad1.20x1.40mm_HandSolder, F.Cu at (56.7, 63.8)
- added R13: 10k, Resistor_SMD:R_0805_2012Metric_Pad1.20x1.40mm_HandSolder, F.Cu at (56.9, 94.6)
- added R14: 10k, Resistor_SMD:R_0805_2012Metric_Pad1.20x1.40mm_HandSolder, F.Cu at (56.8, 83.8)
- added R15: 10k, Resistor_SMD:R_0805_2012Metric_Pad1.20x1.40mm_HandSolder, F.Cu at (55.5, 73.8)
- added R16: 100k, Resistor_SMD:R_0805_2012Metric_Pad1.20x1.40mm_HandSolder, F.Cu at (83.5, 77.2)
- added R17: RVar, Potentiometer_THT:Potentiometer_Bourns_3296W_Vertical, F.Cu at (82.5, 71.8)
- added R18: 10k, Resistor_SMD:R_0805_2012Metric_Pad1.20x1.40mm_HandSolder, F.Cu at (95.0, 70.9)
- added R19: 10k, Resistor_SMD:R_0805_2012Metric_Pad1.20x1.40mm_HandSolder, F.Cu at (89.4, 82.8)
- added R2: 10k, Resistor_SMD:R_0805_2012Metric_Pad1.20x1.40mm_HandSolder, F.Cu at (69.0, 56.6)
- added R20: 56k, Resistor_SMD:R_0805_2012Metric_Pad1.20x1.40mm_HandSolder, F.Cu at (95.5, 78.2)
- added R21: 56k, Resistor_SMD:R_0805_2012Metric_Pad1.20x1.40mm_HandSolder, F.Cu at (99.0, 79.7)
- added R22: 200k, Resistor_SMD:R_0805_2012Metric_Pad1.20x1.40mm_HandSolder, F.Cu at (102.5, 80.7)
- added R23: 100, Resistor_SMD:R_0805_2012Metric_Pad1.20x1.40mm_HandSolder, F.Cu at (171.9, 106.2)
- added R24: 10k, Resistor_SMD:R_0805_2012Metric_Pad1.20x1.40mm_HandSolder, F.Cu at (175.0, 101.1)
- added R27: 0.82k, Resistor_SMD:R_0805_2012Metric_Pad1.20x1.40mm_HandSolder, F.Cu at (119.9, 56.6)
- added R3: 10k, Resistor_SMD:R_0805_2012Metric_Pad1.20x1.40mm_HandSolder, F.Cu at (50.5, 56.9)
- added R33: 0.82k, Resistor_SMD:R_0805_2012Metric_Pad1.20x1.40mm_HandSolder, F.Cu at (115.9, 56.6)
- added R4: 10k, Resistor_SMD:R_0805_2012Metric_Pad1.20x1.40mm_HandSolder, F.Cu at (78.8, 56.5)
- added R44: 10k, Resistor_SMD:R_0805_2012Metric_Pad1.20x1.40mm_HandSolder, F.Cu at (125.5, 68.6)
- added R45: 6.8k, Resistor_SMD:R_0805_2012Metric_Pad1.20x1.40mm_HandSolder, F.Cu at (119.9, 76.2)
- added R46: 6.8k, Resistor_SMD:R_0805_2012Metric_Pad1.20x1.40mm_HandSolder, F.Cu at (115.9, 76.1)
- added R47: 510k 0805, Resistor_SMD:R_0805_2012Metric_Pad1.20x1.40mm_HandSolder, F.Cu at (174.9, 51.3)
- added R48: 510k 0805, Resistor_SMD:R_0805_2012Metric_Pad1.20x1.40mm_HandSolder, F.Cu at (178.4, 51.3)
- added R49: 7.15k 0805, Resistor_SMD:R_0805_2012Metric_Pad1.20x1.40mm_HandSolder, F.Cu at (178.4, 56.3)
- added R5: 100k, Resistor_SMD:R_0805_2012Metric_Pad1.20x1.40mm_HandSolder, F.Cu at (71.4, 87.2)
- added R50: 8.2k, Resistor_SMD:R_0805_2012Metric_Pad1.20x1.40mm_HandSolder, F.Cu at (114.9, 80.0)
- added R51: 10k, Resistor_SMD:R_0805_2012Metric_Pad1.20x1.40mm_HandSolder, F.Cu at (124.9, 73.1)
- added R52: 10k, Resistor_SMD:R_0805_2012Metric_Pad1.20x1.40mm_HandSolder, F.Cu at (124.9, 77.6)
- added R53: 6.8k, Resistor_SMD:R_0805_2012Metric_Pad1.20x1.40mm_HandSolder, F.Cu at (182.9, 55.3)
- added R54: 6.8k, Resistor_SMD:R_0805_2012Metric_Pad1.20x1.40mm_HandSolder, F.Cu at (184.9, 59.8)
- added R55: 8.2k, Resistor_SMD:R_0805_2012Metric_Pad1.20x1.40mm_HandSolder, F.Cu at (182.9, 64.3)
- added R56: 130k 0.5%, Resistor_SMD:R_0805_2012Metric_Pad1.20x1.40mm_HandSolder, F.Cu at (180.4, 67.8)
- added R57: 102k, Resistor_SMD:R_0805_2012Metric_Pad1.20x1.40mm_HandSolder, F.Cu at (166.4, 60.3)
- added R58: 976k, Resistor_SMD:R_0805_2012Metric_Pad1.20x1.40mm_HandSolder, F.Cu at (174.4, 74.8)
- added R59: 360, Resistor_SMD:R_0805_2012Metric_Pad1.20x1.40mm_HandSolder, F.Cu at (168.9, 79.3)
- added R6: RVar, Potentiometer_THT:Potentiometer_Bourns_3296W_Vertical, F.Cu at (70.9, 82.7)
- added R60: 2.2k, Resistor_SMD:R_0805_2012Metric_Pad1.20x1.40mm_HandSolder, F.Cu at (146.5, 71.8)
- added R7: 10k, Resistor_SMD:R_0805_2012Metric_Pad1.20x1.40mm_HandSolder, F.Cu at (76.3, 76.5)
- added R8: 10k, Resistor_SMD:R_0805_2012Metric_Pad1.20x1.40mm_HandSolder, F.Cu at (72.4, 90.7)
- added R9: 56k, Resistor_SMD:R_0805_2012Metric_Pad1.20x1.40mm_HandSolder, F.Cu at (84.4, 87.2)
- added U1: NUCLEO-H503RB, discharger:NUCLEO-H503RB, F.Cu at (127.0, 143.4)
- added U13: INA126U/2K5, Package_SO:SOIC-8_5.3x6.2mm_P1.27mm, F.Cu at (119.4, 68.6)
- added U15: MCP6004, Package_SO:SOIC-14_3.9x8.7mm_P1.27mm, F.Cu at (171.0, 67.8)
- added U16: LTC6992CS6-2-TRMPBF, Package_TO_SOT_SMD:TSOT-23-6, F.Cu at (169.9, 74.9)
- added U17: 6N137, Package_DIP:DIP-8_W7.62mm, F.Cu at (157.8, 77.1)
- added U2: SN74LVC1T45DBV, Package_TO_SOT_SMD:SOT-23-6, F.Cu at (76.9, 154.0)
- added U3: MCP6004, Package_SO:SOIC-14_3.9x8.7mm_P1.27mm, F.Cu at (77.9, 85.7)
- added U4: MCP6004, Package_SO:SOIC-14_3.9x8.7mm_P1.27mm, F.Cu at (89.5, 76.7)
- added U5: CD4052B, Package_SO:TSSOP-16_4.4x5mm_P0.65mm, F.Cu at (66.5, 66.9)
- added U6: VX7805-500, Converter_DCDC:Converter_DCDC_TRACO_TSR0.5-24xx_TSR0.5-24xxx_THT, F.Cu at (101.3, 54.0)
- added U7: ISO1050DUB, Package_SO:SOP-8_6.62x9.15mm_P2.54mm, F.Cu at (72.9, 162.3)
- added U8: MCP6004, Package_SO:SOIC-14_3.9x8.7mm_P1.27mm, F.Cu at (103.3, 71.8)
- added U9: CC1R5-1205SR-E, discharger:CC1R5-1205SR-E, F.Cu at (151.5, 57.3)
Routing:
- net /Temperature Sensor Interface/Temp6_1: track 0.00 -> 38.9 mm
- net Net-(U16-MOD): track 0.00 -> 28.8 mm
- net /Temperature Sensor Interface/Temp3_1: track 0.00 -> 28.8 mm
- net /Temperature Sensor Interface/Temp7_1: track 0.00 -> 28.0 mm
- net Net-(U4B-+): track 0.00 -> 25.9 mm
- net /Temperature Sensor Interface/Temp8_1: track 0.00 -> 24.7 mm
- net /Temperature Sensor Interface/Temp5_1: track 0.00 -> 21.5 mm
- net /Temperature Sensor Interface/Temp4_1: track 0.00 -> 19.9 mm
- net Net-(U3C-+): track 0.00 -> 19.8 mm
- net /Temperature Sensor Interface/Temp1_1: track 0.00 -> 19.8 mm
- net Net-(U8A-+): track 0.00 -> 19.7 mm
- net /Temperature Sensor Interface/Temp2_1: track 0.00 -> 18.2 mm
- net Net-(U4C-+): track 0.00 -> 16.4 mm
- net Net-(U13-+IN): track 0.00 -> 14.0 mm
- net Net-(C30-Pad2): track 0.00 -> 13.7 mm
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- added copper zone on F.Cu, net GND
