File: hardware/gate_driver_daughter_board/gate_driver_daughter_board.kicad_sch (KiCad schematic)
At the start: 0 parts

Commit message: DC/DC added, incomplete Current sense, and incomplete snubber circuit
Parts:
- added C1: C, symbol Device:C
- added C2: 2uF, MKP1848E52010KI2, symbol Device:C
- added C3: 10nF, symbol Device:C
- added C4: 100nF, symbol Device:C
- added C5, C6: 0.1uF, symbol Device:C
- added D1, D2, D3: 1SMB5956BT3G, Diode_SMD:D_SMB, symbol Device:D_Zener
- added D4: D_Schottky, symbol Device:D_Schottky
- added J1, J3: Conn_01x02, symbol Connector_Generic:Conn_01x02
- added J2: Conn_01x08, symbol Connector_Generic:Conn_01x08
- added Q1: CM600HA-28H, symbol Device:Q_NIGBT_CEG
- added R1: R, symbol Device:R
- added R2, Rg: (no value), symbol Device:R
- added Rb: .043, symbol Device:R
- added RpShunt: TBD, symbol Device:R
- added U1: NCD57100DWR2G, Package_SO:SOIC-16W_7.5x10.3mm_P1.27mm, symbol gate_driver_daughter_board:NCD57100DWR2G
- added U2: REC20K-2412SZ, REC20K_RCP, symbol gate_driver_daughter_board:REC20K-2412SZ
- added U3: INA126U/2K5, symbol Amplifier_Instrumentation:INA128
Connections:
- new net: C3.2, C4.2, U1.15 (V_DD1)
- new net: C2.1, D4.1 (K), R2.2
- new net: C2.2, D3.2 (A)
- new net: D1.1 (K), R2.1
- new net: C1.1, R1.2, U1.11 (IN-)
- new net: D1.2 (A), D2.1 (K)
- new net: Q1.1 (C), Rb.1
- new net: J1.1 (Pin_1), Q1.3 (G), U1.4 (OUTH)
- new net: D2.2 (A), D3.1 (K)
- new net: Rg.1, U3.1 (Rg)
- new net: C6.1, U3.4 (V-)
- new net: Rg.2, U3.8 (Rg)
- new net +12V: J2.8 (Pin_8), U2.1 (+VIN)
- new net +12V_Isolated: C5.2, U1.5 (V_DD2), U2.6 (+VOUT), U3.7 (V+)
- new net Battery-: C5.1, C6.2, J1.2 (Pin_2), Q1.2 (E), U1.1 (V_EE2A), U1.3 (GND2), U1.8 (V_EE2), U2.4 (-VOUT), U3.5 (Ref)
- new net GND: C1.2, C4.1, J2.7 (Pin_7), U1.10 (IN+), U1.16 (GND1), U1.9 (GND1A), U2.2 (-VIN)
- new net Rp_CurrShunt+: J3.1 (Pin_1), U3.3 (+)
- new net Rp_CurrShunt-: J3.2 (Pin_2), U3.2 (-)
- new net Rp_CurrentSense: J2.2 (Pin_2)
- new net Rp_GD_Ready: J2.5 (Pin_5), U1.12 (RDY)
- new net Rp_GateDrive: J2.6 (Pin_6), R1.1
- new net ~{Rp_GD_Fault}: J2.3 (Pin_3), U1.13 (~{FLT})
- new net ~{Rp_GD_Reset}: J2.4 (Pin_4), U1.14 (~{RST})
- no-connect marks 0 -> 3
Other:
- note added: "Calibrated Busbar Shunt"
- note added: "Gain roughly in the 30~40 range"
- note added: "Need to find out desat power"
- note added: "Need to test a real shunts resistance to calibrate this."
- note added: "Total Zener Voltage: 600V"
- note added: "Worst Case V(RG) = 250 * 67.7uOhns (Rshunt) = 0.05~"
- note added: "Zener Voltage: 200V"

Commit message: Pre-Testing Changes (Used for Presentation Graphics)
Parts:
- removed C1: C, symbol Device:C
- removed D2, D3: 1SMB5956BT3G, Diode_SMD:D_SMB, symbol Device:D_Zener
- added R3: 1M, symbol Device:R
- added TP1: Snubber+, symbol Connector:TestPoint
- added TP2: Battery-, symbol Connector:TestPoint
- D4: Digikey Link (none) -> https://www.mouser.com/ProductDetail/Toshiba/TRS20H120HS1Q?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; Manufacturer Part Number (none) -> Toshiba
- Rb: value .043 -> 0.43
Connections:
- net Battery-: now also C2.2, D1.2 (A), R3.1, TP2.1
- net GND: now also U1.11 (IN-); no longer U1.10 (IN+)
- net +3.3V: now reaches C3.2, C4.2, U1.15 (V_DD1)
- net at C2.1, D4.1 (K), R2.2: now also R3.2, TP1.1
- net at D4.2 (A): now also Q1.1 (C), Rb.1
- net at R1.2: now also U1.10 (IN+); no longer U1.11 (IN-)
Other:
- note added: "Needs Heatsinking"
- note added: "Snubber Circuit needs a way to dissipate voltage in capacitor without burning it all.."
- note added: "Testpoint to scope and check pulsed voltage in design"
- note removed: "Total Zener Voltage: 600V"
- moved on the sheet: C5, C6, D1, J2, J3, R1, R2, Rb, Rg, RpShunt, U3

Commit message: DC/DC Change
Parts:
- removed C2: 2uF, MKP1848E52010KI2, symbol Device:C
- removed D1: 1SMB5956BT3G, Diode_SMD:D_SMB, symbol Device:D_Zener
- removed J1: Conn_01x02, symbol Connector_Generic:Conn_01x02
- removed R1: R, symbol Device:R
- removed TP1: Snubber+, symbol Connector:TestPoint
- removed TP2: Battery-, symbol Connector:TestPoint
- removed U3: INA126U/2K5, symbol Amplifier_Instrumentation:INA128
- added C10, C20, C7: 100nF, symbol Device:C
- added C11, C18, C8: 10uF, symbol Device:C
- added C12, C13, C14, C15, C16, C17: 1000uF, symbol Device:C_Polarized
- added C19, C9: 1uF, symbol Device:C
- added C25: 0.1uF, symbol Device:C
- added H1: GATE, symbol Mechanical:MountingHole_Pad_MP
- added H2: EMITTER, symbol Mechanical:MountingHole_Pad_MP
- added JP1, JP2, JP3, JP4: Jumper_2_Small_Open, symbol Jumper:Jumper_2_Small_Open
- added R30: 130k 0.5%, symbol Device:R
- added R31: 360, symbol Device:R
- added R32: 2.2k, symbol Device:R
- added R33: 10k, symbol Device:R
- added R36: 102k, symbol Device:R
- added R37: 976k, symbol Device:R
- added R4: R?, Resistor_SMD:R_1206_3216Metric_Pad1.30x1.75mm_HandSolder, symbol Device:R
- added U8: LTC6992CS6-2-TRMPBF, Package_TO_SOT_SMD:TSOT-23-6, symbol discharger:LTC6992CS6-2-TRMPBF
- added U9: 6N137, Package_DIP:DIP-8_W7.62mm, symbol Isolator:6N137
- C3: value 10nF -> 1uF
- D4: value D_Schottky -> VS-QA250FA20; Digikey Link https://www.mouser.com/ProductDetail/Toshiba/TRS20H120HS1Q?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 -> https://www.mouser.com/ProductDetail/Vishay-Semiconductors/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; Digikey Part Number (none) -> 78-VS-QA250FA20; Manufacturer Part Number Toshiba -> Vishay Semiconductors
- Q1, Rb: now fitted
- R2: value (none) -> R?; footprint (none) -> Resistor_SMD:R_1206_3216Metric_Pad1.30x1.75mm_HandSolder; Digikey Link (none) -> https://www.mouser.com/c/passive-components/resistors/film-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
- R3: value 1M -> R?; footprint (none) -> Resistor_SMD:R_1206_3216Metric_Pad1.30x1.75mm_HandSolder; Digikey Link (none) -> https://www.mouser.com/c/passive-components/resistors/film-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
- U2: Digikey Link (none) -> https://www.mouser.com/ProductDetail/RECOM-Power/REC20K-241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
Connections:
- net +12V: now also C10.2, C11.2, C12.1, C13.1, C14.1, C9.2
- net +3.3V: now also R32.1
- net Battery-: now also D4.2 (A), C15.2, C16.2, C17.2, C18.1, C19.1, C20.1, H2.MP, JP4.1 (A); no longer R3.1
- net GND: now also C3.1, C10.1, C11.1, C12.2, C13.2, C14.2, C25.2, C7.1, C8.1, C9.1, R33.1, U9.5 (GND)
- net Rp_GateDrive: now also R4.1
- net at R2.2, R3.2: now also Q1.3 (G), H1.MP, JP3.2 (B); no longer D4.1 (K)
- net at R2.1: now also U1.4 (OUTH)
- net at Q1.1 (C), Rb.1: now also D4.1 (K); no longer D4.2 (A)
- net at U1.10 (IN+): now also R4.2
- net at U1.2 (DESAT): now also JP1.1 (A), JP2.2 (B)
- net at U1.6 (OUTL): now also R3.1
- net at U1.7 (CLAMP): now also JP3.1 (A), JP4.2 (B)
- net +12V_Isolated renamed +15V_Isolated
- net +15V_Isolated: now also C15.1, C16.1, C17.1, C18.2, C19.2, C20.2, C7.2, C8.2, JP1.2 (B)
- new net: R30.1, R37.2, U8.2 (GND)
- new net: R30.2, U8.3 (SET)
- new net: R36.2, R37.1, U8.4 (DIV)
- new net: R31.2, U8.6 (OUT)
- new net: R32.2, U9.6 (VO)
- new net: R31.1, U9.2 (A)
- new net: R33.2, U9.7 (EN)
- new net +5V: C25.1, U9.8 (VCC)
- new net +5V_isolated: R36.1, U8.5 (V+)
- new net HV_-: U9.3 (C)
- no-connect marks 3 -> 5
Other:
- note added: "12V->15V DC/DC"
- note added: "Change R values with testing. Tune to be critically damped. 2-18ohms."
- note added: "Gain roughly in the 60-80 range"
- note added: "High Voltage (Battery Side)"
- note added: "Isolated Gate Driver Chip"
- note added: "Low Voltage"
- note added: "Off-Board"
- note added: "Tune R1 values with testing, because of the unknown Inducatances in system. Limit ripple to 3.3V, damping the system. (1-11 ohms)."
- note removed: "Gain roughly in the 30~40 range"
- note removed: "Need to find out desat power"
- note removed: "Needs Heatsinking"
- note removed: "Snubber Circuit needs a way to dissipate voltage in capacitor without burning it all.."
- note removed: "Testpoint to scope and check pulsed voltage in design"
- note removed: "Zener Voltage: 200V"
- moved on the sheet: C3, C4, C5, C6, D4, J2, J3, Rg, RpShunt, U1

Commit message: Filter Stage Added, Current Gain Stage Added, Simulation Added
Parts:
- removed C3: 1uF, symbol Device:C
- removed C4, C7: 100nF, symbol Device:C
- removed C8: 10uF, symbol Device:C
- removed J2: Conn_01x08, symbol Connector_Generic:Conn_01x08
- added C21: 1uF, Capacitor_SMD:C_0805_2012Metric_Pad1.18x1.45mm_HandSolder, symbol Device:C
- added C22: 10uF, Capacitor_SMD:C_0805_2012Metric_Pad1.18x1.45mm_HandSolder, symbol Device:C
- added C23, C24: 100nF, Capacitor_SMD:C_0805_2012Metric_Pad1.18x1.45mm_HandSolder, symbol Device:C
- added C26: 47nF, Capacitor_SMD:C_0805_2012Metric_Pad1.18x1.45mm_HandSolder, symbol Device:C
- added C27: 10nF, Capacitor_SMD:C_0805_2012Metric_Pad1.18x1.45mm_HandSolder, symbol Device:C
- added C28: 0.33uF, Capacitor_SMD:C_0805_2012Metric_Pad1.18x1.45mm_HandSolder, symbol Device:C
- added C29, C30: 0.1uF, Capacitor_SMD:C_0805_2012Metric_Pad1.18x1.45mm_HandSolder, symbol Device:C
- added C31: 2.2uF, Capacitor_SMD:C_0805_2012Metric_Pad1.18x1.45mm_HandSolder, symbol Device:C
- added J1: Conn_01x07, Connector_Molex:Molex_Nano-Fit_105309-xx07_1x07_P2.50mm_Vertical, symbol Connector_Generic:Conn_01x07
- added R38, R39, R41, R42, R43, R44: 6.8k, symbol Device:R
- added R40: 8.2k, symbol Device:R
- added U3: INA821xD, Package_SO:SOIC-8_3.9x4.9mm_P1.27mm, symbol Amplifier_Instrumentation:INA821xD
- added U4: MCP6004, symbol Amplifier_Operational:MCP6004
- added U5: LM7805_TO220, Package_TO_SOT_THT:TO-220-3_Vertical, symbol Regulator_Linear:LM7805_TO220
- added U6: LF33_TO220, Package_TO_SOT_THT:TO-220-3_Vertical, symbol Regulator_Linear:LF33_TO220
- C10, C11, C18, C19, C20, C25, C5, C9: footprint (none) -> Capacitor_SMD:C_0805_2012Metric_Pad1.18x1.45mm_HandSolder
- C12, C13, C14, C15, C16, C17: footprint (none) -> gate_driver_daughter_board:25V1000uF
- J3: footprint (none) -> Connector_Molex:Molex_Nano-Fit_105309-xx02_1x02_P2.50mm_Vertical
- JP1, JP2, JP3, JP4: footprint (none) -> Connector_PinHeader_2.54mm:PinHeader_1x02_P2.54mm_Vertical
- Rg: value (none) -> 549
- RpShunt1: renamed from RpShunt; value TBD -> 30u
- U2: footprint REC20K_RCP -> (none)
- renumbered Rb to Rb1
Connections:
- net +12V: now also C30.2, J1.7 (Pin_7), U6.1 (VI)
- net +15V_Isolated: now also C22.2, C23.2, C28.2, U5.1 (VI); no longer C5.2
- net +3.3V: now also C21.2, C24.2, C31.2, J1.1 (Pin_1), U6.3 (VO)
- net Battery-: now also R30.1, R37.2, U8.2 (GND), C26.1, C28.1, C29.1, R42.2, U3.6 (Ref), U4.11 (V-), U4.3 (+), U5.2 (GND)
- net GND: now also C21.1, C22.1, C23.1, C24.1, C30.1, C31.1, J1.6 (Pin_6), U6.2 (GND)
- net Rp_CurrShunt+: now also U3.1 (-)
- net Rp_CurrShunt-: now also U3.4 (+)
- net Rp_GD_Ready: now also J1.4 (Pin_4)
- net Rp_GateDrive: now also J1.5 (Pin_5)
- net ~{Rp_GD_Fault}: now also J1.2 (Pin_2)
- net ~{Rp_GD_Reset}: now also J1.3 (Pin_3)
- net at U8.1 (MOD): now also R41.2, U4.7
- net at JP2.1 (A): now also JP1.1 (A), U1.2 (DESAT)
- net at JP4.2 (B), U1.7 (CLAMP): now also JP3.2 (B); no longer JP3.1 (A)
- net at H1.MP, Q1.3 (G), R2.2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: now also JP3.1 (A); no longer JP3.2 (B)
- net at C6.1: now also U3.5 (Vs-)
- net +120V, Battery: now reaches Rb1.2
- net at Rg.1: now also U3.2 (Rg)
- net at Rg.2: now also U3.3 (Rg)
- net +5V_isolated renamed +5V_Isolated
- net +5V_Isolated: now also C5.2, C29.2, R44.2, U3.8 (Vs+), U4.4 (V+), U5.3 (VO)
- new net: C27.2, R40.2, R43.1, U4.1
- new net: R43.2, R44.1, U4.5 (+)
- new net: C26.2, R38.1, R39.2, R40.1
- new net: R39.1, U3.7
- new net: R41.1, R42.1, U4.6 (-)
- new net: C27.1, R38.2, U4.2 (-)
- now unconnected: JP2.2 (B)
- no-connect marks 5 -> 11
Other:
- note added: "Amplification, Bias and Gain Calculations: https://www.desmos.com/calculator/qjhpey8gnn"
- note added: "Filter Simulation"
- note added: "G = 1 * ((49.4*10^3)/Rg) G = 1 * ((40.4*10^3)/549) = 89.98~"
- note removed: "Calibrated Busbar Shunt"
- note removed: "Gain roughly in the 60-80 range"
- note removed: "Need to test a real shunts resistance to calibrate this."
- note removed: "Worst Case V(RG) = 250 * 67.7uOhns (Rshunt) = 0.05~"
- moved on the sheet: C10, C11, C12, C25, C5, C6, C9, D4, H1, H2, J3, JP1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

Commit message: Final Schematic Changes, Footprints assigned, ready for review / layout
Parts:
- removed C6: 0.1uF, symbol Device:C
- removed JP1, JP2: Jumper_2_Small_Open, Connector_PinHeader_2.54mm:PinHeader_1x02_P2.54mm_Vertical, symbol Jumper:Jumper_2_Small_Open
- removed R33: 10k, symbol Device:R
- removed R41, R42, R43, R44: 6.8k, symbol Device:R
- added C15, C23, C28: 0.1uF, Capacitor_SMD:C_0805_2012Metric_Pad1.18x1.45mm_HandSolder, symbol Device:C
- added C27: 0.33uF, Capacitor_SMD:C_0805_2012Metric_Pad1.18x1.45mm_HandSolder, symbol Device:C
- added R10: 1k, Resistor_SMD:R_0805_2012Metric_Pad1.20x1.40mm_HandSolder, symbol Device:R
- added R11: 154k, Resistor_SMD:R_0805_2012Metric_Pad1.20x1.40mm_HandSolder, symbol Device:R
- added R12, R17, R18: 10k, Resistor_SMD:R_0805_2012Metric_Pad1.20x1.40mm_HandSolder, symbol Device:R
- added R13: 8.87k, Resistor_SMD:R_0805_2012Metric_Pad1.20x1.40mm_HandSolder, symbol Device:R
- added TP1: InAmp_Bias/Amp, TestPoint:TestPoint_Pad_D3.0mm, symbol Connector:TestPoint
- added TP2: InAmp_Filtered, symbol Connector:TestPoint
- added TP3: InAmpOut, symbol Connector:TestPoint
- added U9: LM7805_TO220, Package_TO_SOT_THT:TO-220-3_Vertical, symbol Regulator_Linear:LM7805_TO220
- R14: renamed from R40; footprint (none) -> Resistor_SMD:R_0805_2012Metric_Pad1.20x1.40mm_HandSolder
- R15: renamed from R38; footprint (none) -> Resistor_SMD:R_0805_2012Metric_Pad1.20x1.40mm_HandSolder
- R16: renamed from R39; footprint (none) -> Resistor_SMD:R_0805_2012Metric_Pad1.20x1.40mm_HandSolder
- R3: renamed from R32; footprint (none) -> Resistor_SMD:R_0805_2012Metric_Pad1.20x1.40mm_HandSolder
- R4: renamed from R31; footprint (none) -> Resistor_SMD:R_0805_2012Metric_Pad1.20x1.40mm_HandSolder
- R5: renamed from R36; footprint (none) -> Resistor_SMD:R_0805_2012Metric_Pad1.20x1.40mm_HandSolder
- R6: renamed from R37; footprint (none) -> Resistor_SMD:R_0805_2012Metric_Pad1.20x1.40mm_HandSolder
- R7: renamed from R30; footprint (none) -> Resistor_SMD:R_0805_2012Metric_Pad1.20x1.40mm_HandSolder
- Rg1: renamed from Rg; footprint (none) -> Resistor_SMD:R_0805_2012Metric_Pad1.20x1.40mm_HandSolder
- RpShunt1: now fitted
- U2: footprint (none) -> gate_driver_daughter_board:REC20K_RCP
- U7: renamed from U4; footprint (none) -> Package_SO:SOIC-14_3.9x8.7mm_P1.27mm
- U8: renamed from U3; value INA821xD -> INA826
- renumbered C12 to C1, C21 to C10, C25 to C11, C23 to C12, C22 to C13, C15 to C14, C28 to C18, C18 to C19, C30 to C2, C19 to C20, C20 to C21, C29 to C22, C27 to C24, C26 to C25, C5 to C26, C13 to C3, C14 to C4, C31 to C5, C11 to C6, C9 to C7, C10 to C8, C24 to C9, D4 to D1, J3 to J2, JP4 to JP1, JP3 to JP2, R4 to R1, R2 to R8, R3 to R9, U6 to U1, U9 to U3, U1 to U4, U8 to U5, U5 to U6
Connections:
- net HV_- is gone; now on net Battery-: U3.3 (C)
- net +12V: now also C27.2, U9.1 (VI)
- net +15V_Isolated: now also U4.2 (DESAT)
- net +3.3V: no longer J1.1 (Pin_1)
- net +5V: now also U3.7 (EN)
- net +5V_Isolated: now also C15.1, C23.2, R12.2, R17.2
- net Battery-: now also RpShunt1.1, RpShunt1.2, U8.5 (Vs-), C15.2, C23.1, C27.1, C28.1, R13.1, R18.1, U9.2 (GND); no longer U8.6 (Ref)
- net at U5.1 (MOD), U7.7: now also R10.2, TP1.1
- net at C24.2, R14.2, U7.1: now also U7.5 (+), TP2.1
- net at R16.1, U8.7: now also TP3.1
- net at U7.6 (-): now also R10.1, R11.2
- net Rp_CurrentSense: now reaches R3.2, U3.6 (VO)
- net Rp_CurrentSense: now also J1.1 (Pin_1)
- net at U7.12 (+): now also R12.1, R13.2
- net at U7.13 (-): now also U7.14, R11.1
- net at U7.10 (+): now also R17.1, R18.2
- net at U7.8: now also U7.9 (-), U8.6 (Ref)
- new net 5V: C28.2, U9.3 (VO)
- no-connect marks 11 -> 4
Other:
- note added: "2.35V~"
- note added: "2.5V"
- note added: "2.5VRef"
- note added: "Amplification, Bias and Gain Calculations: https://www.desmos.com/calculator/3htui5wwul Amplification / Bias Correction Stage: Vout ~= (Vin*1.0065) + 2.366 Vin(min): 2.5V -> Vout(min): 0.15V Vin(max): 3.175V -> Vout(max): 0.829V"
- note added: "Desaturation check will be done externally. Will add auxillary components if time permits"
- note added: "Filtering Stage (Click for Simulation) 1kHz Cutoff Freq, MFB Topology, Butterworth"
- note added: "In-Amp Stage: G = 1 * ((49.4*10^3)/Rg) G = 1 * ((40.4*10^3)/549) = 89.98~ Vout = (Vin * Gain (89.98)) + Vref(2.5V) Vin(min): 0V -> Vout(min): 2.5V Vin(max): 0.0075V -> Vout(max): 3.175V"
- note added: "Isolated ADC Design copied from main board"
- note added: "V = I * R V = 265 * 30 * 10^-6 = 0.00795V 0.3uV / A (RpShunt is a Calibrated Busbar)"
- note removed: "Amplification, Bias and Gain Calculations: https://www.desmos.com/calculator/qjhpey8gnn"
- note removed: "Filter Simulation"
- note removed: "G = 1 * ((49.4*10^3)/Rg) G = 1 * ((40.4*10^3)/549) = 89.98~"
- moved on the sheet: C11, C24, C25, C26, D1, J2, Q1, R14, R15, R16, R3, R4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

Commit message: PCBrev1
Parts:
- removed J1: Conn_01x07, Connector_Molex:Molex_Nano-Fit_105309-xx07_1x07_P2.50mm_Vertical, symbol Connector_Generic:Conn_01x07
- added J1: Conn_01x08, Connector_Molex:Molex_Nano-Fit_105309-xx08_1x08_P2.50mm_Vertical, symbol Connector_Generic:Conn_01x08
- added J3: Conn_01x02, Connector_Molex:Molex_Nano-Fit_105309-xx02_1x02_P2.50mm_Vertical, symbol Connector_Generic:Conn_01x02
- added R19: 100k, Resistor_SMD:R_0805_2012Metric_Pad1.20x1.40mm_HandSolder, symbol Device:R
- H1, H2: footprint (none) -> gate_driver_daughter_board:MountingHole_4.3x6.2mm_M4_Pad
- TP2: footprint (none) -> TestPoint:TestPoint_Pad_D3.0mm
- TP3: footprint (none) -> TestPoint:TestPoint_Pad_2.0x2.0mm
- renumbered RpShunt1 to RbShunt1
Connections:
- net 5V is gone; now on net +5V: C28.2, U9.3 (VO)
- net +12V: now also J1.1 (Pin_1)
- net Battery-: now also C12.1, C13.1, U7.10 (+); no longer C27.1, C28.1, U7.3 (+), U9.2 (GND)
- net GND: now also C27.1, C28.1, U9.2 (GND), J1.2 (Pin_2), R19.1; no longer C12.1, C13.1
- net Rp_CurrentSense: now also J1.3 (Pin_3)
- net Rp_GD_Ready: now also J1.5 (Pin_5)
- net ~{Rp_GD_Fault}: now also J1.6 (Pin_6)
- net at R17.1, R18.2: now also U7.12 (+); no longer U7.10 (+)
- net at R14.2, TP2.1, U7.5 (+): now also C24.1, U7.8; no longer C24.2, U7.1
- net at U7.13 (-), U7.14: now also U8.6 (Ref); no longer R11.1
- net at R12.1, R13.2: now also U7.3 (+); no longer U7.12 (+)
- net Rp_CurrShunt+ renamed Rb_CurrShunt+
- net Rp_CurrShunt- renamed Rb_CurrShunt-
- net Rp_GateDrive renamed Rb_GateDrive
- net Rb_GateDrive: now also J1.4 (Pin_4)
- net ~{Rp_GD_Reset} renamed ~{Rp_GD_ResetFinal}
- net ~{Rp_GD_ResetFinal}: now also J1.8 (Pin_8), J3.2 (Pin_2), R19.2
- new net: R11.1, U7.1, U7.2 (-)
- new net: C24.2, R15.2, U7.9 (-)
- new net ~{Rb_GD_Reset}: J1.7 (Pin_7), J3.1 (Pin_1)
Other:
- note added: "OverTempSwitch IN"
- note added: "OverTempSwitch OUT"
- moved on the sheet: C24, U7A, U7C, U7D
